File: boards/demi1/demiurge-panel_template.kicad_pcb (KiCad board)
At the start: 2 copper layers, 40.4 x 128.5 mm, 23 parts

Commit message: Filled background in drawings.
Other:
- board text added: "USB"
Changed lines of the file:
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@@
+    (effects (font (size 2 2) (thickness 0.3)) (justify mirror))
+  )
+  (gr_text "USB" (at 81.5 63.1) (layer "B.SilkS")
     (effects (font (size 2 2) (thickness 0.3)) (justify mirror))
   )
