File: boards/demi1/demiurge-panel_template.kicad_pcb (KiCad board)
At the start: 2 copper layers, 40.4 x 128.5 mm, 23 parts

Commit message: Work on the build system and not be dependent on MounRiver.
Parts:
- added G***: LOGO, LOGO, B.Cu at (96.7, 52.6)
Other:
- board text removed: "Awesome Audio Apparatus"
