File: boards/demi1/demiurge.kicad_sch (KiCad schematic)
At the start: 155 parts, among them J12 Micro_SD_Card_Det_Hirose_DM3AT, J2 Conn_01x06, U1 MCP6002, U10 TL072, U11 TL072, U13 STM32F446, U2 AMS1117-3.3, U3 MCP6002, U4 AW20036, U5 W25Q128JVS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

Commit message: wrong file names on RevG photos.
Parts:
- added C? (x4): 100nF, Capacitor_SMD:C_0603_1608Metric, symbol Device:C
- added R?: 10k, Resistor_SMD:R_0603_1608Metric, symbol Device:R
Connections:
- net -12V: now also C?.2, C?.2, C?.2, C?.2; no longer C18.2, C20.2, C22.2, C24.2
- net GND: now also R?.2
- net GNDA: now also C18.2, C20.2, C22.2, C24.2, C?.1, C?.1, C?.1, C?.1
- net at D9.3, R28.2, U6.4 (B): now also R?.1
Other:
- moved on the sheet: C18, C20, C22, C24
